Commit message: Update URDF sensor placements to match physical robot
- Sonar (HC-SR04): moved from chassis front to wrist_link, 3cm above
  gripper mount — enables scanning by sweeping the arm
- IR sensors: moved to rear of chassis facing backward as parking
  sensors, 4cm off floor, just inside tracks
- Body motion sensor: added body_motion_link on Pi at rear, lying flat
  with module arrow pointing right (yaw -90deg from forward)

https://claude.ai/code/session_01BD1jEJCFRd5ttdPPtLv2bq

File: src/argos_description/urdf/argos.urdf.xacro (robot description, xacro)
@@ -25,16 +25,16 @@
   <xacro:property name="imu_y"     value="0.0"   />
   <xacro:property name="imu_z"     value="0.050" />
-  <xacro:property name="sonar_x"   value="0.120" />
-  <xacro:property name="sonar_y"   value="0.0"   />
-  <xacro:property name="sonar_z"   value="0.040" />
+  <!-- sonar is now arm-mounted (on wrist, above gripper) — offset below -->
+  <xacro:property name="sonar_wrist_z" value="0.030" />
   <xacro:property name="camera_x"  value="0.110" />
   <xacro:property name="camera_y"  value="0.0"   />
   <xacro:property name="camera_z"  value="0.090" />
-  <xacro:property name="ir1_x"     value="0.125" />
+  <!-- IR sensors face rearward (parking sensors), just inside tracks -->
+  <xacro:property name="ir1_x"     value="-0.115"/>
   <xacro:property name="ir1_y"     value="-0.060"/>
-  <xacro:property name="ir1_z"     value="0.020" />
-  <xacro:property name="ir2_x"     value="0.125" />
+  <xacro:property name="ir1_z"     value="0.008" />
+  <xacro:property name="ir2_x"     value="-0.115"/>
   <xacro:property name="ir2_y"     value="0.060" />
-  <xacro:property name="ir2_z"     value="0.020" />
+  <xacro:property name="ir2_z"     value="0.008" />
   <!-- arm base is at rear-centre of chassis top -->
   <xacro:property name="arm_base_x" value="-0.060" />
@@ -131,5 +131,6 @@
     <origin xyz="${imu_x} ${imu_y} ${track_radius + chassis_height + imu_z}" rpy="0 0 0" />
   </joint>
-  <!-- Sonar (HC-SR04) — front of chassis -->
+  <!-- Sonar (HC-SR04) — mounted on wrist, above gripper attachment -->
+  <!-- Moves with the arm so it can scan by sweeping joints -->
   <link name="sonar_link">
     <visual>
@@ -142,7 +143,8 @@
   </link>
   <joint name="sonar_joint" type="fixed">
-    <parent link="base_link" />
+    <parent link="wrist_link" />
     <child link="sonar_link" />
-    <origin xyz="${sonar_x} ${sonar_y} ${track_radius + sonar_z}" rpy="0 0 0" />
+    <!-- 3 cm above wrist origin, pointing along the wrist/gripper axis -->
+    <origin xyz="0 0 ${sonar_wrist_z}" rpy="0 0 0" />
   </joint>
   <!-- Camera — front-top of chassis -->
@@ -167,5 +169,5 @@
     <origin xyz="0 0 0" rpy="${-pi/2} 0 ${-pi/2}" />
   </joint>
-  <!-- IR sensors — front corners -->
+  <!-- IR sensors — rear-facing parking sensors, just inside tracks -->
   <xacro:macro name="ir_sensor" params="name x y z">
     <link name="${name}_link">
@@ -181,5 +183,6 @@
       <parent link="base_link" />
       <child link="${name}_link" />
-      <origin xyz="${x} ${y} ${track_radius + z}" rpy="0 0 0" />
+      <!-- facing rearward (pi yaw), low to ground -->
+      <origin xyz="${x} ${y} ${track_radius + z}" rpy="0 0 ${pi}" />
     </joint>
   </xacro:macro>
@@ -337,4 +340,24 @@
   </joint>
   <!-- ================================================================== -->
+  <!-- Body-mounted motion sensor (Flotilla LSM303D on Raspberry Pi)      -->
+  <!-- Flat on Pi at rear of chassis, arrow silkscreen pointing right     -->
+  <!-- (module X axis = robot -Y), so yaw -90°                           -->
+  <!-- ================================================================== -->
+  <link name="body_motion_link">
+    <visual>
+      <geometry>
+        <box size="0.015 0.015 0.003" />
+      </geometry>
+      <material name="green" />
+    </visual>
+  </link>
+  <joint name="body_motion_joint" type="fixed">
+    <parent link="base_link" />
+    <child link="body_motion_link" />
+    <!-- rear of chassis, on top of Pi, lying flat, arrow pointing right -->
+    <origin xyz="-0.080 0 ${track_radius + chassis_height + 0.005}"
+            rpy="0 0 ${-pi/2}" />
+  </joint>
+  <!-- ================================================================== -->
   <!-- Arm-mounted motion sensor (Flotilla LSM303D on elbow link)         -->
   <!-- ================================================================== -->

Commit message: Fix URDF arm and camera placement to match physical robot
- Move arm base from rear to front-centre of chassis
- Move camera from front-centre to side of chassis towards rear,
  facing forward with arm in view

https://claude.ai/code/session_01BD1jEJCFRd5ttdPPtLv2bq

File: src/argos_description/urdf/argos.urdf.xacro (robot description, xacro)
@@ -27,7 +27,7 @@
   <!-- sonar is now arm-mounted (on wrist, above gripper) — offset below -->
   <xacro:property name="sonar_wrist_z" value="0.030" />
-  <xacro:property name="camera_x"  value="0.110" />
-  <xacro:property name="camera_y"  value="0.0"   />
-  <xacro:property name="camera_z"  value="0.090" />
+  <xacro:property name="camera_x"  value="-0.060" />
+  <xacro:property name="camera_y"  value="0.085"  />
+  <xacro:property name="camera_z"  value="0.090"  />
   <!-- IR sensors face rearward (parking sensors), just inside tracks -->
   <xacro:property name="ir1_x"     value="-0.115"/>
@@ -37,7 +37,7 @@
   <xacro:property name="ir2_y"     value="0.060" />
   <xacro:property name="ir2_z"     value="0.008" />
-  <!-- arm base is at rear-centre of chassis top -->
-  <xacro:property name="arm_base_x" value="-0.060" />
-  <xacro:property name="arm_base_y" value="0.0"    />
+  <!-- arm base is at front-centre of chassis top -->
+  <xacro:property name="arm_base_x" value="0.060" />
+  <xacro:property name="arm_base_y" value="0.0"   />
   <xacro:property name="arm_base_z" value="${chassis_height / 2}" />
   <!-- ================================================================== -->
@@ -148,5 +148,5 @@
     <origin xyz="0 0 ${sonar_wrist_z}" rpy="0 0 0" />
   </joint>
-  <!-- Camera — front-top of chassis -->
+  <!-- Camera — side of chassis towards rear, facing forward -->
   <link name="camera_link">
     <visual>
